File: hardware/reDIP-sx.sch (KiCad schematic (older format))
At the start: 81 parts, among them J1 DX07S016JA3, J10 Conn_01x01, J2 Conn_01x01, J3 Conn_01x01, J4 Conn_01x01, J5 Conn_01x06, J6 Conn_01x06, J7 Conn_01x10, J8 Conn_01x10, J9 Conn_01x01, Q1 PEMH4, Q2 PDTA143ZMB, U1 NCP163AFCT120T2G, U10 CBTD3306GT, U11 SN74CBTD16211DGVR, U2 NCP167AFCT330T2G, U3 FSA221UMX, U4 SGTL5000XNLA3, U5 ESP32-PICO-V3-02, U6 CP2102N-A02-GQFN24, U7 FSA8049UCX, U8 ICE40UP5K-SG48I, U9 APS6404L-3SQR-SN

Commit message: Usability and manufacturability improvements
* Swapped pins for 3V3 and AO2
* Replaced 0.35mm pitch BGA LDOs with larger pitch parts, improved layout
* Removed IO2 pullup
* Added solder pad for RGB LED strip
* Increased solder mask clearance
* Updated silk screen
Parts:
- removed R12: 2.2k, Resistor_SMD:R_0201_0603Metric, symbol Device:R
- added J2: Conn_01x01, reDIP:SolderWirePad_1x01_SMD_1x2mm, symbol Connector_Generic:Conn_01x01
- U1: value NCP163AFCT120T2G -> NCP163AMX120TBG; footprint ONSemi:WLCSP-4_0.64x0.64mm_Layout2x2_P0.35mm -> ONSemi:CASE711AJ_1.0x1.0mm_P0.65mm; symbol ONSemi:NCP163AFCT120T2G -> ONSemi:NCP163AMX120TBG; Description IC REG LDO 1.2V 250mA WLCSP-4 -> IC REG LDO 1.2V 250mA XDFN4; PN NCP163AFCT120T2G -> NCP163AMX120TBG
- U2: value NCP167AFCT330T2G -> NCP167AMX330TBG; footprint ONSemi:WLCSP-4_0.64x0.64mm_Layout2x2_P0.35mm -> ONSemi:CASE711AJ_1.0x1.0mm_P0.65mm; symbol ONSemi:NCP167AFCT330T2G -> ONSemi:NCP167AMX330TBG; Description IC REG LDO 3.3V 700mA WLCSP-4 -> IC REG LDO 3.3V 700mA XDFN4; PN NCP167AFCT330T2G -> NCP167AMX330TBG
- renumbered J9 to J10, J10 to J11, J2 to J3, J3 to J4, J4 to J5, J5 to J6, J6 to J7, J7 to J8, J8 to J9
Connections:
- net +1V2: now also U1.1 (OUT), U2.3 (EN); no longer U1.A2 (OUT), U2.B1 (EN)
- net +3V3: now also J7.1 (Pin_1), U2.1 (OUT); no longer J7.3 (Pin_3), U2.A2 (OUT)
- net +5V: now also U1.3 (EN), U1.4 (IN), U2.4 (IN); no longer U1.A1 (IN), U1.B1 (EN), U2.A1 (IN)
- net AUDIO_OUT_2: now also J7.3 (Pin_3); no longer J7.1 (Pin_1)
- net GND: now also U1.2 (GND), U2.2 (GND); no longer U1.B2 (GND), U2.B2 (GND)
- net LED_DO: now reaches D5.1 (DO)
- net LED_DO: now also J2.1 (Pin_1)
- no-connect marks 22 -> 21
Other:
- note added: "To mount in a SID socket; use a\n28 pin stamped DIP socket with pins\n1 - 4 and 28 removed as an adapter.\n\nWarning! Pin 28 in a SID socket must\nNOT be connected (Vdd: +9V / +12V)!"
- note removed: "To mount in a SID socket; use a\n28 pin stamped DIP socket with pins\n1 - 4 and 28 removed as an adapter.\n\nWarning! The 3.3V output must\nNOT be connected to pin 28\nin a SID socket (Vdd: +9V / +12V)!"
- moved on the sheet: C30, D4, D5, Q2, R11

Commit message: A few small improvements
* Added SPI SCLK source termination for iCE40UP5K
* Changed R11 to 100Ω
* Changed C27 to 0.1µF
* Replaced a few capacitors with more readily available parts
* Added datasheet URLs for all parts
Parts:
- added R12: 22, Resistor_SMD:R_0201_0603Metric, symbol Device:R_Small
- C1, C3: Description CAP CER 2.2uF 10V 10% X6S 0402 -> CAP CER 2.2uF 16V 10% X6S 0402; PN GRM155C81A225KE11D -> GRM155C81C225KE11D
- C10, C15: Description CAP CER 0.1uF 10V 10% X6S 0201 -> CAP CER 0.22uF 6.3V 20% X5R 0201; Notes 1.55V DC AUDIO -> 1.55V DC AUDIO DERATED TO 0.1uF; PN GRM033C81A104KE14D -> GRM033R60J224KE15D
- C27: value 1uF -> 0.1uF; Description CAP CER 4.7uF 6.3V 20% X5R 0201 -> CAP CER 0.22uF 6.3V 20% X5R 0201; Notes 3.3V DC DERATED TO 1uF -> 3.3V DC DERATED TO 0.1uF; PN GRM035R60J475ME15D -> GRM033R60J224KE15D
- R11: value 330 -> 100; Description RES 330Ω 50mW 5% 0201 -> RES 100Ω 50mW 5% 0201; PN ERJ-1GNJ331C -> ERJ-1GNJ101C
- renumbered J3 to J2, J4 to J3, J5 to J4, J6 to J5, J7 to J6, J8 to J7, J9 to J8, J2 to J9
Connections:
- net SPI_SCLK: now also R12.2; no longer U8.15 (IOB_34a_SPI_SCK)
- new net: R12.1, U8.15 (IOB_34a_SPI_SCK)
Other:
- moved on the sheet: J10, J11, J9

Commit message: Usability and manufacturability improvements
* Increased minimum via size (good luck on increasing it further!)
* Corrected footprint rotation for D3 (IPC-7351)
* Removed split in stencil apertures for pin-in-paste
* Changed to shorter pin USB-C receptacle, yielding improved hole
  fill for partial pin penetration soldering
* Adjustments to fab and silk screen layers
* Added alternative ESP32 APLL configuration example to schematic
Parts:
- J1: value DX07S016JA3 -> DX07S016JA1; footprint JAE:USB_C_Receptacle_JAE_DX07S016JA3_PinInPaste -> JAE:USB_C_Receptacle_JAE_DX07S016JA1; PN DX07S016JA3R1500 -> DX07S016JA1R1500
Other:
- note added: "24.575996MHz:\nsdm0 = 149\nsdm1 = 212\nsdm2 = 5\nodiv = 6"
- note added: "24.576009MHz:\nsdm0 = 40\nsdm1 = 15\nsdm2 = 7\nodiv = 7"
- note added: "Example APLL clock frequency\n24.576MHz (512 * 48kHz):"
- note added: "To mount in a SID socket; Remove pins 1 - 4\nand 28 from a 28 pin stamped DIP socket,\nand use this as an adapter.\n\nWarning! AUDIO_OUT_2 must NOT be connected\nto pin 28 in a SID socket (Vdd: +9V / +12V)!"
- note removed: "Example APLL clock frequency\n24.576MHz (512 * 48kHz):\n\nsdm0 = 149\nsdm1 = 212\nsdm2 = 5\nodiv = 6"
- note removed: "To mount in a SID socket; use a\n28 pin stamped DIP socket with pins\n1 - 4 and 28 removed as an adapter.\n\nWarning! Pin 28 in a SID socket must\nNOT be connected (Vdd: +9V / +12V)!"
Changed lines of the file:
@@
 Sheet 1 1
 Title "reDIP sx"
-Date "2020-12-31"
+Date "2021-01-17"
 Rev "0.1"
 Comp "Nimrod"
-Comment1 "© 2020 Dag Lem"
+Comment1 "© 2020 - 2021 Dag Lem"
 Comment2 "Licensed under CERN-OHL-S v2 (https://ohwr.org/cern_ohl_s_v2.txt)"
 Comment3 ""
@@
 NoConn ~ 3250 8750
 Text Notes 4400 7650 0    50   ~ 0
-To mount in a SID socket; use a\n28 pin stamped DIP socket with pins\n1 - 4 and 28 removed as an adapter.\n\nWarning! Pin 28 in a SID socket must\nNOT be connected (Vdd: +9V / +12V)!
+To mount in a SID socket; Remove pins 1 - 4\nand 28 from a 28 pin stamped DIP socket,\nand use this as an adapter.\n\nWarning! AUDIO_OUT_2 must NOT be connected\nto pin 28 in a SID socket (Vdd: +9V / +12V)!
 $Comp
 L FPGA_Lattice:ICE40UP5K-SG48ITR U8
@@
 P 1400 4550
 F 0 "J1" H 1400 5450 50  0000 C CNN
-F 1 "DX07S016JA3" H 1400 5350 50  0000 C CNN
-F 2 "JAE:USB_C_Receptacle_JAE_DX07S016JA3_PinInPaste" H 1550 4550 50  0001 C CNN
-F 3 "https://www.jae.com/en/connectors/series/detail/product/id=91781" H 1550 4550 50  0001 C CNN
+F 1 "DX07S016JA1" H 1400 5350 50  0000 C CNN
+F 2 "JAE:USB_C_Receptacle_JAE_DX07S016JA1" H 1550 4550 50  0001 C CNN
+F 3 "https://www.jae.com/en/connectors/series/detail/product/id=91780" H 1550 4550 50  0001 C CNN
 F 4 "Japan Aviation Electronics Industry, Ltd." H 1400 4550 50  0001 C CNN "Mfg"
-F 5 "DX07S016JA3R1500" H 1400 4550 50  0001 C CNN "PN"
+F 5 "DX07S016JA1R1500" H 1400 4550 50  0001 C CNN "PN"
 F 6 "CONN USB-C" H 1400 4550 50  0001 C CNN "Description"
 	1    1400 4550
@@
 Wire Wire Line
 	10350 10250 10600 10250
-Text Notes 8000 5700 0    50   ~ 0
-Example APLL clock frequency\n24.576MHz (512 * 48kHz):\n\nsdm0 = 149\nsdm1 = 212\nsdm2 = 5\nodiv = 6
+Text Notes 8000 5250 0    50   ~ 0
+Example APLL clock frequency\n24.576MHz (512 * 48kHz):
 Wire Wire Line
 	7300 10250 7550 10250
@@
 Wire Wire Line
 	10350 10150 10250 10150
+Text Notes 8000 5700 0    50   ~ 0
+24.575996MHz:\nsdm0 = 149\nsdm1 = 212\nsdm2 = 5\nodiv = 6
+Text Notes 8700 5700 0    50   ~ 0
+24.576009MHz:\nsdm0 = 40\nsdm1 = 15\nsdm2 = 7\nodiv = 7
 $EndSCHEMATC
